Commit message: added joint limits for arm group

File: snacbot_description/urdf/snacbot.urdf (robot description, URDF)
Before this commit: robot snacbot, 11 links, 10 joints
Joints:
- joint elbow_joint: limit (none) -> lower=-1.5 upper=1.6 effort=300 velocity=4.01; type continuous -> revolute
- joint palm_joint: limit (none) -> lower=-1.6 upper=1.6 effort=300 velocity=4.01; type continuous -> revolute
- joint shoulder_joint: limit (none) -> lower=-1.85 upper=1.85 effort=300 velocity=4.01; type continuous -> revolute
- joint waist_joint: limit (none) -> lower=-3.14 upper=3.14 effort=300 velocity=4.01; type continuous -> revolute
- joint wrist_joint: limit (none) -> lower=-1.6 upper=1.85 effort=300 velocity=4.01; type continuous -> revolute

File: snacbot_description/urdf/snacbot.xacro (robot description, xacro)
@@ -192,15 +192,17 @@
   <child link="base_link" />
 </joint>
-<joint name="waist_joint" type="continuous">
+<joint name="waist_joint" type="revolute">
   <origin xyz="0.0 0.0 0.073675" rpy="0 0 0"/>
   <parent link="base_link"/>
   <child link="shoulder_link"/>
   <axis xyz="0.0 0.0 1.0"/>
-</joint>
-<joint name="shoulder_joint" type="continuous">
+  <limit lower="-3.14" upper="3.14" effort="300" velocity="4.01" />
+</joint>
+<joint name="shoulder_joint" type="revolute">
   <origin xyz="0.0 -0.009 0.04" rpy="0 0 0"/>
   <parent link="shoulder_link"/>
   <child link="arm_link"/>
   <axis xyz="0.0 1.0 0.0"/>
+  <limit lower="-1.85" upper="1.85" effort="300" velocity="4.01" />
 </joint>
 <joint name="shoulder_shadow_joint" type="continuous">
@@ -211,21 +213,24 @@
   <mimic joint="shoulder_joint" multiplier="-1" offset="0" />
 </joint>
-<joint name="elbow_joint" type="continuous">
+<joint name="elbow_joint" type="revolute">
   <origin xyz="0.027 -0.011075 0.2042" rpy="0 0 0"/>
   <parent link="arm_link"/>
   <child link="forearm_link"/>
   <axis xyz="0.0 -1.0 0.0"/>
-</joint>
-<joint name="wrist_joint" type="continuous">
+  <limit lower="-1.5" upper="1.6" effort="300" velocity="4.01" />
+</joint>
+<joint name="wrist_joint" type="revolute">
   <origin xyz="0.1808 0.000425 0.0125" rpy="0 0 0"/>
   <parent link="forearm_link"/>
   <child link="hand_link"/>
   <axis xyz="-0.0 -1.0 0.0"/>
-</joint>
-<joint name="palm_joint" type="continuous">
+  <limit lower="-1.6" upper="1.85" effort="300" velocity="4.01" />
+</joint>
+<joint name="palm_joint" type="revolute">
   <origin xyz="0.06531 0.0201 -5e-05" rpy="0 0 0"/>
   <parent link="hand_link"/>
   <child link="palm_link"/>
   <axis xyz="1.0 0.0 0.0"/>
+  <limit lower="-1.6" upper="1.6" effort="300" velocity="4.01" />
 </joint>
 <joint name="gripper_joint" type="continuous">

Commit message: working gripper

File: snacbot_description/urdf/snacbot.urdf (robot description, URDF)
Before this commit: robot snacbot, 11 links, 10 joints
Links:
- added link ee_link
Joints:
- added joint ee_joint: type fixed, parent palm_link, child ee_link, origin xyz=0.126 0.0 0.0 rpy=0 0 0
- joint finger1_joint: mimic (none) -> joint=gripper_joint multiplier=0.33 offset=0
- joint finger2_joint: mimic (none) -> joint=gripper_joint multiplier=-0.33 offset=0
- joint gripper_joint: limit (none) -> lower=0.26 upper=2.6 effort=300 velocity=4.01; type continuous -> revolute

File: snacbot_description/urdf/snacbot.xacro (robot description, xacro)
@@ -188,4 +188,7 @@
   </collision>
 </link>
+<link name="ee_link">
+  <origin xyz="0 0 0" rpy="0 0 0"/>
+</link>
 <joint name="base_joint" type="fixed">
   <parent link="world" />
@@ -234,9 +237,10 @@
   <limit lower="-1.6" upper="1.6" effort="300" velocity="4.01" />
 </joint>
-<joint name="gripper_joint" type="continuous">
+<joint name="gripper_joint" type="revolute">
   <origin xyz="0.04704 0.000306 -0.0208" rpy="0 0 0"/>
   <parent link="palm_link"/>
   <child link="gripper_driving_link"/>
   <axis xyz="-0.0 -0.0 1.0"/>
+  <limit lower="0.26" upper="2.6" effort="300" velocity="4.01" />
 </joint>
 <joint name="finger1_joint" type="continuous">
@@ -245,4 +249,5 @@
   <child link="finger1_link"/>
   <axis xyz="0.0 0.0 -1.0"/>
+  <mimic joint="gripper_joint" multiplier="0.33" offset="0" />
 </joint>
 <joint name="finger2_joint" type="continuous">
@@ -251,4 +256,10 @@
   <child link="finger2_link"/>
   <axis xyz="0.0 0.0 -1.0"/>
+  <mimic joint="gripper_joint" multiplier="-0.33" offset="0" />
+</joint>
+<joint name="ee_joint" type="fixed">
+  <origin xyz="0.126 0.0 0.0" rpy="0 0 0"/>
+  <parent link="palm_link"/>
+  <child link="ee_link"/>
 </joint>
 </robot>

Commit message: added realsense to urdf

File: snacbot_description/urdf/snacbot.urdf (robot description, URDF)
Before this commit: robot snacbot, 12 links, 11 joints
Links:
- added link camera_bottom_screw_frame
- added link camera_link, mass 0.072; collision box size=0.02505 0.09 0.025; visual mesh filename=package://realsense2_description/meshes/d435.dae
Joints:
- added joint camera_joint: type fixed, parent palm_link, child camera_bottom_screw_frame, origin xyz=0 0 0 rpy=0 0 0
- added joint camera_link_joint: type fixed, parent camera_bottom_screw_frame, child camera_link, origin xyz=0.010600000000000002 0.0175 0.0125 rpy=0 0 0

File: snacbot_description/urdf/snacbot.xacro (robot description, xacro)
@@ -4,4 +4,6 @@
 <xacro:include filename="$(find snacbot_description)/urdf/snacbot.trans" />
 <xacro:include filename="$(find snacbot_description)/urdf/snacbot.gazebo" />
+<xacro:arg name="use_nominal_extrinsics" default="false" />
+<xacro:include filename="$(find realsense2_description)/urdf/_d435i.urdf.xacro"/>
 <link name="world"/>
 <link name="base_link">
@@ -128,4 +130,7 @@
   </collision>
 </link>
+<xacro:sensor_d435i parent="palm_link" use_nominal_extrinsics="$(arg use_nominal_extrinsics)">
+  <origin xyz="0.04 0 0.035" rpy="0 0 0"/>
+</xacro:sensor_d435i>
 <link name="gripper_driving_link">
   <inertial>

Commit message: urdf realsense fix

File: snacbot_description/urdf/snacbot.urdf (robot description, URDF)
Before this commit: robot snacbot, 14 links, 13 joints
Joints:
- joint camera_joint: origin xyz=0 0 0 rpy=0 0 0 -> xyz=0.04 0 0.035 rpy=0 0 0

Commit message: update urdf

File: snacbot_description/urdf/snacbot.urdf (robot description, URDF)
Before this commit: robot snacbot, 14 links, 13 joints
Joints:
- joint ee_joint: origin xyz=0.126 0.0 0.0 rpy=0 0 0 -> xyz=0.126 0.0 0.007 rpy=0 0 0
- joint palm_joint: limit lower=-1.6 upper=1.6 effort=300 velocity=4.01 -> lower=-3.14 upper=3.14 effort=300 velocity=4.01

File: snacbot_description/urdf/snacbot.xacro (robot description, xacro)
@@ -241,5 +241,5 @@
     <child link="palm_link"/>
     <axis xyz="1.0 0.0 0.0"/>
-    <limit lower="-1.6" upper="1.6" effort="300" velocity="4.01" />
+    <limit lower="-3.14" upper="3.14" effort="300" velocity="4.01" />
   </joint>
   <joint name="gripper_joint" type="revolute">
@@ -265,5 +265,5 @@
   </joint>
   <joint name="ee_joint" type="fixed">
-    <origin xyz="0.126 0.0 0.0" rpy="0 0 0"/>
+    <origin xyz="0.126 0.0 0.007" rpy="0 0 0"/>
     <parent link="palm_link"/>
     <child link="ee_link"/>

File: snacbot_description/urdf/snacbot_ik.urdf (robot description, URDF)
Before this commit: robot snacbot, 11 links, 10 joints
Links:
- added link camera_bottom_screw_frame
- added link camera_link, mass 0.072; collision box size=0.02505 0.09 0.025; visual mesh filename=package://realsense2_description/meshes/d435.dae
Joints:
- added joint camera_joint: type fixed, parent palm_link, child camera_bottom_screw_frame, origin xyz=0.04 0 0.035 rpy=0 0 0
- added joint camera_link_joint: type fixed, parent camera_bottom_screw_frame, child camera_link, origin xyz=0.010600000000000002 0.0175 0.0125 rpy=0 0 0
- joint ee_joint: origin xyz=0.126 0.0 0.0 rpy=0 0 0 -> xyz=0.126 0.0 0.007 rpy=0 0 0
- joint palm_joint: limit lower=-1.6 upper=1.6 effort=300 velocity=4.01 -> lower=-3.14 upper=3.14 effort=300 velocity=4.01
